File: outputs.kicad_sch (KiCad schematic)
At the start: 8 parts

Commit message: changed I2C temp sensor to thermistor
Connections:
- net ADC_1 renamed ADC_MOTOR_CURRENT_1
- net ADC_2 renamed ADC_MOTOR_CURRENT_2
- net ADC_3 renamed ADC_MOTOR_CURRENT_3
- net ADC_4 renamed ADC_MOTOR_CURRENT_4
Changed lines of the file:
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@@
 		)
 	)
-	(global_label "ADC_1"
+	(global_label "ADC_MOTOR_CURRENT_1"
 		(shape input)
 		(at 127 40.64 0)
@@
 		)
 		(property "Intersheetrefs" "${INTERSHEET_REFS}"
-			(at 135.7909 40.64 0)
+			(at 152.6637 40.64 0)
 			(hide yes)
 			(show_name no)
@@
 		)
 	)
-	(global_label "ADC_3"
+	(global_label "ADC_MOTOR_CURRENT_3"
 		(shape input)
 		(at 255.27 43.18 0)
@@
 		)
 		(property "Intersheetrefs" "${INTERSHEET_REFS}"
-			(at 264.0609 43.18 0)
+			(at 280.9337 43.18 0)
 			(hide yes)
 			(show_name no)
@@
 		)
 	)
-	(global_label "ADC_2"
+	(global_label "ADC_MOTOR_CURRENT_2"
 		(shape input)
 		(at 127 100.33 0)
@@
 		)
 		(property "Intersheetrefs" "${INTERSHEET_REFS}"
-			(at 135.7909 100.33 0)
+			(at 152.6637 100.33 0)
 			(hide yes)
 			(show_name no)
@@
 		)
 	)
-	(global_label "ADC_4"
+	(global_label "ADC_MOTOR_CURRENT_4"
 		(shape input)
 		(at 255.27 100.33 0)
@@
 		)
 		(property "Intersheetrefs" "${INTERSHEET_REFS}"
-			(at 264.0609 100.33 0)
+			(at 280.9337 100.33 0)
 			(hide yes)
 			(show_name no)

Commit message: Placed designators
Parts:
- renumbered C58 to C50, C59 to C51, C40 to C52, C49 to C53, D35 to D21, D29 to D22, D34 to D23, D32 to D24
Changed lines of the file:
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@@
 		(dnp no)
 		(fields_autoplaced yes)
-		(property "Reference" "C58"
+		(property "Reference" "C50"
 			(at 254 48.2599 0)
 			(show_name no)
@@
 			(project "ADC_Board"
 				(path "/1c5d070a-ffd0-423b-a405-f3ed0dbc8144"
-					(reference "C58")
+					(reference "C50")
 					(unit 1)
 				)
@@
 		(dnp no)
 		(fields_autoplaced yes)
-		(property "Reference" "C40"
+		(property "Reference" "C52"
 			(at 125.73 45.7199 0)
 			(show_name no)
@@
 			(project "ADC_Board"
 				(path "/1c5d070a-ffd0-423b-a405-f3ed0dbc8144"
-					(reference "C40")
+					(reference "C52")
 					(unit 1)
 				)
@@
 		(dnp no)
 		(fields_autoplaced yes)
-		(property "Reference" "#PWR0135"
+		(property "Reference" "#PWR070"
 			(at 250.19 62.23 0)
 			(hide yes)
@@
 			(project "ADC_Board"
 				(path "/1c5d070a-ffd0-423b-a405-f3ed0dbc8144"
-					(reference "#PWR0135")
+					(reference "#PWR070")
 					(unit 1)
 				)
@@
 		(dnp no)
 		(fields_autoplaced yes)
-		(property "Reference" "#PWR0100"
+		(property "Reference" "#PWR065"
 			(at 121.92 30.48 0)
 			(hide yes)
@@
 			(project "ADC_Board"
 				(path "/1c5d070a-ffd0-423b-a405-f3ed0dbc8144"
-					(reference "#PWR0100")
+					(reference "#PWR065")
 					(unit 1)
 				)
@@
 		(dnp no)
 		(fields_autoplaced yes)
-		(property "Reference" "D29"
+		(property "Reference" "D22"
 			(at 124.46 31.4324 90)
 			(show_name no)
@@
 			(project "ADC_Board"
 				(path "/1c5d070a-ffd0-423b-a405-f3ed0dbc8144"
-					(reference "D29")
+					(reference "D22")
 					(unit 1)
 				)
@@
 		(dnp no)
 		(fields_autoplaced yes)
-		(property "Reference" "C59"
+		(property "Reference" "C51"
 			(at 125.73 105.4099 0)
 			(show_name no)
@@
 			(project "ADC_Board"
 				(path "/1c5d070a-ffd0-423b-a405-f3ed0dbc8144"
-					(reference "C59")
+					(reference "C51")
 					(unit 1)
 				)
@@
 		(dnp no)
 		(fields_autoplaced yes)
-		(property "Reference" "#PWR0136"
+		(property "Reference" "#PWR067"
 			(at 121.92 90.17 0)
 			(hide yes)
@@
 			(project "ADC_Board"
 				(path "/1c5d070a-ffd0-423b-a405-f3ed0dbc8144"
-					(reference "#PWR0136")
+					(reference "#PWR067")
 					(unit 1)
 				)
@@
 		(dnp no)
 		(fields_autoplaced yes)
-		(property "Reference" "#PWR0122"
+		(property "Reference" "#PWR072"
 			(at 250.19 119.38 0)
 			(hide yes)
@@
 			(project "ADC_Board"
 				(path "/1c5d070a-ffd0-423b-a405-f3ed0dbc8144"
-					(reference "#PWR0122")
+					(reference "#PWR072")
 					(unit 1)
 				)
@@
 		(dnp no)
 		(fields_autoplaced yes)
-		(property "Reference" "#PWR0134"
+		(property "Reference" "#PWR069"
 			(at 250.19 33.02 0)
 			(hide yes)
@@
 			(project "ADC_Board"
 				(path "/1c5d070a-ffd0-423b-a405-f3ed0dbc8144"
-					(reference "#PWR0134")
+					(reference "#PWR069")
 					(unit 1)
 				)
@@
 		(dnp no)
 		(fields_autoplaced yes)
-		(property "Reference" "C49"
+		(property "Reference" "C53"
 			(at 254 105.4099 0)
 			(show_name no)
@@
 			(project "ADC_Board"
 				(path "/1c5d070a-ffd0-423b-a405-f3ed0dbc8144"
-					(reference "C49")
+					(reference "C53")
 					(unit 1)
 				)
@@
 		(dnp no)
 		(fields_autoplaced yes)
-		(property "Reference" "#PWR0101"
+		(property "Reference" "#PWR066"
 			(at 121.92 59.69 0)
 			(hide yes)
@@
 			(project "ADC_Board"
 				(path "/1c5d070a-ffd0-423b-a405-f3ed0dbc8144"
-					(reference "#PWR0101")
+					(reference "#PWR066")
 					(unit 1)
 				)
@@
 		(dnp no)
 		(fields_autoplaced yes)
-		(property "Reference" "#PWR0117"
+		(property "Reference" "#PWR071"
 			(at 250.19 90.17 0)
 			(hide yes)
@@
 			(project "ADC_Board"
 				(path "/1c5d070a-ffd0-423b-a405-f3ed0dbc8144"
-					(reference "#PWR0117")
+					(reference "#PWR071")
 					(unit 1)
 				)
@@
 		(dnp no)
 		(fields_autoplaced yes)
-		(property "Reference" "D35"
+		(property "Reference" "D21"
 			(at 124.46 91.1224 90)
 			(show_name no)
@@
 			(project "ADC_Board"
 				(path "/1c5d070a-ffd0-423b-a405-f3ed0dbc8144"
-					(reference "D35")
+					(reference "D21")
 					(unit 1)
 				)
@@
 		(dnp no)
 		(fields_autoplaced yes)
-		(property "Reference" "#PWR0137"
+		(property "Reference" "#PWR068"
 			(at 121.92 119.38 0)
 			(hide yes)
@@
 			(project "ADC_Board"
 				(path "/1c5d070a-ffd0-423b-a405-f3ed0dbc8144"
-					(reference "#PWR0137")
+					(reference "#PWR068")
 					(unit 1)
 				)
@@
 		(dnp no)
 		(fields_autoplaced yes)
-		(property "Reference" "D34"
+		(property "Reference" "D23"
 			(at 252.73 33.9724 90)
 			(show_name no)
@@
 			(project "ADC_Board"
 				(path "/1c5d070a-ffd0-423b-a405-f3ed0dbc8144"
-					(reference "D34")
+					(reference "D23")
 					(unit 1)
 				)
@@
 		(dnp no)
 		(fields_autoplaced yes)
-		(property "Reference" "D32"
+		(property "Reference" "D24"
 			(at 252.73 91.1224 90)
 			(show_name no)
@@
 			(project "ADC_Board"
 				(path "/1c5d070a-ffd0-423b-a405-f3ed0dbc8144"
-					(reference "D32")
-					(unit 1)
-				)
+					(reference "D24")
+					(unit 1)
+				)
