File: ADC_Board.kicad_sch (KiCad schematic)
At the start: 50 parts, among them J7 Wire_Solder_2Pin, J9 Conn_01x07_Socket, Q4 DOD40P03, SW1 SW_Push, U1 TPS70933DBVR, U2 STM32G030K6Tx, Y1 HSO321S 16MHZ 3.3V

Commit message: changed I2C temp sensor to thermistor
Parts:
- removed R21, R22: 4.7k, Resistor_SMD:R_0603_1608Metric_Pad0.98x0.95mm_HandSolder, symbol Device:R
Connections:
- net ADC_THERMISTOR_1: now reaches U2.14 (PA7)
- net ADC_THERMISTOR_2: now reaches U2.16 (PB1)
- net ADC_THERMISTOR_3: now reaches U2.17 (PB2)
- net ADC_THERMISTOR_4: now reaches U2.31 (PB7)
- net ADC_1 renamed ADC_MOTOR_CURRENT_1
- net ADC_2 renamed ADC_MOTOR_CURRENT_2
- net ADC_3 renamed ADC_MOTOR_CURRENT_3
- net ADC_4 renamed ADC_MOTOR_CURRENT_4
- net I2C_SCL renamed ADC_THERMISTOR_5
- net I2C_SDA renamed ADC_THERMISTOR_6
Other:
- moved on the sheet: C4, C6, C8, C9, D2, D20, D21, D22, D23, D24, D25, D26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

Commit message: Placed designators
Parts:
- renumbered C29 to C13, C17 to C21, C16 to C23, C6 to C44, C8 to C47, C9 to C48, C4 to C49, C32 to C5, C31 to C9, D23 to D12, D22 to D13, D21 to D14, D27 to D15, D20 to D16, D25 to D17, D2 to D18, D24 to D19, D26 to D20, D1 to D5, D12 to D7, D13 to D9, F4 to F3, H3 to H2, H2 to H3, H1 to H4, J7 to J1, J9 to J4, R12 to R23, R35 to R24, R38 to R27, R83 to R52, R82 to R53, R81 to R54, R80 to R55, R79 to R56, R10 to R57, R50 to R61, R49 to R62, R48 to R63, R54 to R64, R51 to R65, R53 to R66, R9 to R67, U2 to U12, U1 to U6

Commit message: generated production files
Parts:
- added TP10, TP11, TP12, TP13, TP9: TestPoint, TestPoint:TestPoint_Pad_1.0x1.0mm, symbol Connector:TestPoint
- R23, R24, R27: now not fitted
- SW1: LCSC Part # C318884 -> C93157
Connections:
- net at U12.1 (PB9): now also TP12.1
- net at U12.20 (PC6): now also TP10.1
- net at U12.26 (PA15): now also TP9.1
- net at U12.3 (PC15): now also TP11.1
- net at U12.32 (PB8): now also TP13.1

Commit message: Fixed DNP parts on BOM
Parts:
- R23, R24, R27: now fitted
Changed lines of the file:
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@@
 		(on_board yes)
 		(in_pos_files yes)
-		(dnp yes)
+		(dnp no)
 		(fields_autoplaced yes)
 		(property "Reference" "R24"
@@
 		(on_board yes)
 		(in_pos_files yes)
-		(dnp yes)
+		(dnp no)
 		(fields_autoplaced yes)
 		(property "Reference" "R23"
@@
 		(on_board yes)
 		(in_pos_files yes)
-		(dnp yes)
+		(dnp no)
 		(fields_autoplaced yes)
 		(property "Reference" "R27"
