File: pwm_driver.kicad_sch (KiCad schematic)
At the start: 16 parts, among them U8 SN74HCS08PWR, U9 SN74HCS02PWR

Commit message: Placed designators
Parts:
- renumbered C25 to C32, C28 to C35, C23 to C36, C26 to C38, C27 to C39, C24 to C40, R84 to R36, R86 to R37, R31 to R40, R27 to R41, R85 to R44, R28 to R46, R29 to R48, R87 to R49, U8 to U11
Changed lines of the file:
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@@
 		(dnp no)
 		(fields_autoplaced yes)
-		(property "Reference" "#PWR069"
+		(property "Reference" "#PWR038"
 			(at 71.12 74.93 0)
 			(hide yes)
@@
 			(project "ADC_Board"
 				(path "/a6998454-3219-43c5-85ea-b974e718b0de"
-					(reference "#PWR069")
+					(reference "#PWR038")
 					(unit 1)
 				)
@@
 		(in_pos_files yes)
 		(dnp no)
-		(property "Reference" "R87"
+		(property "Reference" "R49"
 			(at 240.792 80.01 90)
 			(show_name no)
@@
 			(project "ADC_Board"
 				(path "/a6998454-3219-43c5-85ea-b974e718b0de"
-					(reference "R87")
+					(reference "R49")
 					(unit 1)
 				)
@@
 		(dnp no)
 		(fields_autoplaced yes)
-		(property "Reference" "#PWR0140"
+		(property "Reference" "#PWR048"
 			(at 237.49 80.01 0)
 			(hide yes)
@@
 			(project "ADC_Board"
 				(path "/a6998454-3219-43c5-85ea-b974e718b0de"
-					(reference "#PWR0140")
+					(reference "#PWR048")
 					(unit 1)
 				)
@@
 		(dnp no)
 		(fields_autoplaced yes)
-		(property "Reference" "U8"
+		(property "Reference" "U11"
 			(at 144.78 119.38 0)
 			(show_name no)
@@
 			(project "ADC_Board"
 				(path "/a6998454-3219-43c5-85ea-b974e718b0de"
-					(reference "U8")
+					(reference "U11")
 					(unit 1)
 				)
@@
 		(dnp no)
 		(fields_autoplaced yes)
-		(property "Reference" "C28"
+		(property "Reference" "C35"
 			(at 74.93 60.9599 0)
 			(show_name no)
@@
 			(project "ADC_Board"
 				(path "/a6998454-3219-43c5-85ea-b974e718b0de"
-					(reference "C28")
+					(reference "C35")
 					(unit 1)
 				)
@@
 		(dnp no)
 		(fields_autoplaced yes)
-		(property "Reference" "#PWR068"
+		(property "Reference" "#PWR041"
 			(at 120.65 154.94 0)
 			(hide yes)
@@
 			(project "ADC_Board"
 				(path "/a6998454-3219-43c5-85ea-b974e718b0de"
-					(reference "#PWR068")
+					(reference "#PWR041")
 					(unit 1)
 				)
@@
 		(dnp no)
 		(fields_autoplaced yes)
-		(property "Reference" "#PWR067"
+		(property "Reference" "#PWR040"
 			(at 120.65 100.33 0)
 			(hide yes)
@@
 			(project "ADC_Board"
 				(path "/a6998454-3219-43c5-85ea-b974e718b0de"
-					(reference "#PWR067")
+					(reference "#PWR040")
 					(unit 1)
 				)
@@
 		(dnp no)
 		(fields_autoplaced yes)
-		(property "Reference" "#PWR0138"
+		(property "Reference" "#PWR037"
 			(at 52.07 77.47 0)
 			(hide yes)
@@
 			(project "ADC_Board"
 				(path "/a6998454-3219-43c5-85ea-b974e718b0de"
-					(reference "#PWR0138")
+					(reference "#PWR037")
 					(unit 1)
 				)
@@
 		(dnp no)
 		(fields_autoplaced yes)
-		(property "Reference" "#PWR0139"
+		(property "Reference" "#PWR049"
 			(at 238.76 48.26 0)
 			(hide yes)
@@
 			(project "ADC_Board"
 				(path "/a6998454-3219-43c5-85ea-b974e718b0de"
-					(reference "#PWR0139")
+					(reference "#PWR049")
 					(unit 1)
 				)
@@
 		(dnp no)
 		(fields_autoplaced yes)
-		(property "Reference" "C26"
+		(property "Reference" "C38"
 			(at 214.63 97.7899 0)
 			(show_name no)
@@
 			(project "ADC_Board"
 				(path "/a6998454-3219-43c5-85ea-b974e718b0de"
-					(reference "C26")
+					(reference "C38")
 					(unit 1)
 				)
@@
 		(in_pos_files yes)
 		(dnp no)
-		(property "Reference" "R31"
+		(property "Reference" "R40"
 			(at 60.96 56.642 90)
 			(show_name no)
@@
 			(project "ADC_Board"
 				(path "/a6998454-3219-43c5-85ea-b974e718b0de"
-					(reference "R31")
+					(reference "R40")
 					(unit 1)
 				)
@@
 		(in_pos_files yes)
 		(dnp no)
-		(property "Reference" "R29"
+		(property "Reference" "R48"
 			(at 60.96 90.932 90)
 			(show_name no)
@@
 			(project "ADC_Board"
 				(path "/a6998454-3219-43c5-85ea-b974e718b0de"
-					(reference "R29")
+					(reference "R48")
 					(unit 1)
 				)
@@
 		(dnp no)
 		(fields_autoplaced yes)
-		(property "Reference" "#PWR050"
+		(property "Reference" "#PWR047"
 			(at 219.71 83.82 0)
 			(hide yes)
@@
 			(project "ADC_Board"
 				(path "/a6998454-3219-43c5-85ea-b974e718b0de"
-					(reference "#PWR050")
+					(reference "#PWR047")
 					(unit 1)
 				)
@@
 		(dnp no)
 		(fields_autoplaced yes)
-		(property "Reference" "C25"
+		(property "Reference" "C32"
 			(at 175.26 58.4199 0)
 			(show_name no)
@@
 			(project "ADC_Board"
 				(path "/a6998454-3219-43c5-85ea-b974e718b0de"
-					(reference "C25")
+					(reference "C32")
 					(unit 1)
 				)
@@
 		(in_pos_files yes)
 		(dnp no)
-		(property "Reference" "R84"
+		(property "Reference" "R36"
 			(at 55.372 43.18 90)
 			(show_name no)
@@
 			(project "ADC_Board"
 				(path "/a6998454-3219-43c5-85ea-b974e718b0de"
-					(reference "R84")
+					(reference "R36")
 					(unit 1)
 				)
@@
 		(in_pos_files yes)
 		(dnp no)
-		(property "Reference" "R28"
+		(property "Reference" "R46"
 			(at 228.6 93.472 90)
 			(show_name no)
@@
 			(project "ADC_Board"
 				(path "/a6998454-3219-43c5-85ea-b974e718b0de"
-					(reference "R28")
+					(reference "R46")
 					(unit 1)
 				)
@@
 		(dnp no)
 		(fields_autoplaced yes)
-		(property "Reference" "#PWR0133"
+		(property "Reference" "#PWR036"
 			(at 52.07 43.18 0)
 			(hide yes)
@@
 			(project "ADC_Board"
 				(path "/a6998454-3219-43c5-85ea-b974e718b0de"
-					(reference "#PWR0133")
+					(reference "#PWR036")
 					(unit 1)
 				)
@@
 		(dnp no)
 		(fields_autoplaced yes)
-		(property "Reference" "#PWR052"
+		(property "Reference" "#PWR039"
 			(at 71.12 109.22 0)
 			(hide yes)
@@
 			(project "ADC_Board"
 				(path "/a6998454-3219-43c5-85ea-b974e718b0de"
-					(reference "#PWR052")
+					(reference "#PWR039")
 					(unit 1)
 				)
@@
 		(in_pos_files yes)
 		(dnp no)
-		(property "Reference" "R27"
+		(property "Reference" "R41"
 			(at 229.87 61.722 90)
 			(show_name no)
@@
 			(project "ADC_Board"
 				(path "/a6998454-3219-43c5-85ea-b974e718b0de"
-					(reference "R27")
+					(reference "R41")
 					(unit 1)
 				)
@@
 		(dnp no)
 		(fields_autoplaced yes)
-		(property "Reference" "#PWR066"
+		(property "Reference" "#PWR044"
 			(at 182.88 53.34 0)
 			(hide yes)
@@
 			(project "ADC_Board"
 				(path "/a6998454-3219-43c5-85ea-b974e718b0de"
-					(reference "#PWR066")
+					(reference "#PWR044")
 					(unit 1)
 				)
@@
 		(dnp no)
 		(fields_autoplaced yes)
-		(property "Reference" "C24"
+		(property "Reference" "C40"
 			(at 175.26 113.0299 0)
 			(show_name no)
@@
 			(project "ADC_Board"
 				(path "/a6998454-3219-43c5-85ea-b974e718b0de"
-					(reference "C24")
+					(reference "C40")
 					(unit 1)
 				)
@@
 		(dnp no)
 		(fields_autoplaced yes)
-		(property "Reference" "#PWR065"
+		(property "Reference" "#PWR045"
 			(at 182.88 107.95 0)
 			(hide yes)
@@
 			(project "ADC_Board"
 				(path "/a6998454-3219-43c5-85ea-b974e718b0de"
-					(reference "#PWR065")
+					(reference "#PWR045")
 					(unit 1)
 				)
@@
 		(dnp no)
 		(fields_autoplaced yes)
-		(property "Reference" "C27"
+		(property "Reference" "C39"
 			(at 74.93 95.2499 0)
 			(show_name no)
@@
 			(project "ADC_Board"
 				(path "/a6998454-3219-43c5-85ea-b974e718b0de"
-					(reference "C27")
+					(reference "C39")
 					(unit 1)
 				)
@@
 		(in_pos_files yes)
 		(dnp no)
-		(property "Reference" "R86"
+		(property "Reference" "R37"
 			(at 242.062 48.26 90)
 			(show_name no)
@@
 			(project "ADC_Board"
 				(path "/a6998454-3219-43c5-85ea-b974e718b0de"
-					(reference "R86")
+					(reference "R37")
 					(unit 1)
 				)
@@
 		(dnp no)
 		(fields_autoplaced yes)
-		(property "Reference" "C23"
+		(property "Reference" "C36"
 			(at 215.9 69.8499 0)
 			(show_name no)
@@
 			(project "ADC_Board"
 				(path "/a6998454-3219-43c5-85ea-b974e718b0de"
-					(reference "C23")
+					(reference "C36")
 					(unit 1)
 				)
@@
 		(dnp no)
 		(fields_autoplaced yes)
-		(property "Reference" "#PWR063"
+		(property "Reference" "#PWR043"
 			(at 171.45 127 0)
 			(hide yes)
@@
 			(project "ADC_Board"
 				(path "/a6998454-3219-43c5-85ea-b974e718b0de"
-					(reference "#PWR063")
+					(reference "#PWR043")
 					(unit 1)
 				)
@@
 		(in_pos_files yes)
 		(dnp no)
-		(property "Reference" "R85"
+		(property "Reference" "R44"
 			(at 55.372 77.47 90)
 			(show_name no)
@@
 			(project "ADC_Board"
 				(path "/a6998454-3219-43c5-85ea-b974e718b0de"
-					(reference "R85")
+					(reference "R44")
 					(unit 1)
 				)
@@
 		(dnp no)
 		(fields_autoplaced yes)
-		(property "Reference" "#PWR051"
+		(property "Reference" "#PWR046"
 			(at 218.44 111.76 0)
 			(hide yes)
@@
 			(project "ADC_Board"
 				(path "/a6998454-3219-43c5-85ea-b974e718b0de"
-					(reference "#PWR051")
+					(reference "#PWR046")
 					(unit 1)
 				)
@@
 		(dnp no)
 		(fields_autoplaced yes)
-		(property "Reference" "#PWR064"
+		(property "Reference" "#PWR042"
 			(at 171.45 72.39 0)
 			(hide yes)
@@
 			(project "ADC_Board"
 				(path "/a6998454-3219-43c5-85ea-b974e718b0de"
-					(reference "#PWR064")
-					(unit 1)
-				)
+					(reference "#PWR042")
+					(unit 1)
+				)

Commit message: generated production files
Parts:
- R36, R37, R44, R49: now not fitted
Changed lines of the file:
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@@
 		(on_board yes)
 		(in_pos_files yes)
-		(dnp no)
+		(dnp yes)
 		(property "Reference" "R49"
 			(at 240.792 80.01 90)
@@
 		(on_board yes)
 		(in_pos_files yes)
-		(dnp no)
+		(dnp yes)
 		(property "Reference" "R36"
 			(at 55.372 43.18 90)
@@
 		(on_board yes)
 		(in_pos_files yes)
-		(dnp no)
+		(dnp yes)
 		(property "Reference" "R37"
 			(at 242.062 48.26 90)
@@
 		(on_board yes)
 		(in_pos_files yes)
-		(dnp no)
+		(dnp yes)
 		(property "Reference" "R44"
 			(at 55.372 77.47 90)

Commit message: Fixed DNP parts on BOM
Parts:
- R36, R37, R44, R49: now fitted
Changed lines of the file:
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@@
 		(on_board yes)
 		(in_pos_files yes)
-		(dnp yes)
+		(dnp no)
 		(property "Reference" "R49"
 			(at 240.792 80.01 90)
@@
 		(on_board yes)
 		(in_pos_files yes)
-		(dnp yes)
+		(dnp no)
 		(property "Reference" "R36"
 			(at 55.372 43.18 90)
@@
 		(on_board yes)
 		(in_pos_files yes)
-		(dnp yes)
+		(dnp no)
 		(property "Reference" "R37"
 			(at 242.062 48.26 90)
@@
 		(on_board yes)
 		(in_pos_files yes)
-		(dnp yes)
+		(dnp no)
 		(property "Reference" "R44"
 			(at 55.372 77.47 90)
